File: src/hardware/AuxPower.kicad_pcb (KiCad board)
At the start: 2 copper layers, 90 x 90 mm, 104 parts, among them J1 MC 1,5/2, J10 MC 1,5/4, J11 S3B-XH-A, J12 S3B-XH-A, J13 S3B-XH-A, J14 S3B-XH-A, J15 S3B-XH-A, J16 B3B-XH-A, J17 B4B-XH-A, J2 MC 1,5/2, J3 MC 1,5/2, J4 MC 1,5/2, J5 MC 1,5/2, J6 MC 1,5/4, J7 MC 1,5/4, J8 MC 1,5/4, J9 MC 1,5/4, K1 AQZ202G, K2 AQZ202G, K3 AQZ202G, K4 AQZ202G, K5 AQZ202G, U1 ZXCT1009, U2 ZXCT1009, U3 ZXCT1009, U4 ZXCT1009, U5 ZXCT1009, U6 PIC18F26K83, U7 PI4IOE5V6416, U8 MCP9701

Commit message: Added I2C resistor marking
Other:
- board text added: "I2C"
Changed lines of the file:
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@@
 	)
 	(gr_line
+		(start 30.95 76.05)
+		(end 30.95 76.35)
+		(stroke
+			(width 0.2)
+			(type solid)
+		)
+		(layer "B.SilkS")
+	)
+	(gr_line
+		(start 34.85 76.05)
+		(end 34.85 76.35)
+		(stroke
+			(width 0.2)
+			(type solid)
+		)
+		(layer "B.SilkS")
+	)
+	(gr_line
+		(start 30.95 76.05)
+		(end 34.85 76.05)
+		(stroke
+			(width 0.2)
+			(type solid)
+		)
+		(layer "B.SilkS")
+	)
+	(gr_line
 		(start 75 40)
 		(end 75 105)
@@
 		)
 	)
+	(gr_text "I2C"
+		(at 32.9 75.8 0)
+		(layer "B.SilkS")
+		(effects
+			(font
+				(size 1 0.8)
+				(thickness 0.2)
+				(bold yes)
+			)
+			(justify bottom mirror)
+		)
+	)
 	(gr_text "1"
 		(at 23 103 0)
@@
 		)
 	)
+	(group ""
+		(members "47d75d72-ee19-4c6b-8a22-f7c86566f7c9" "6db72c65-edac-42c8-8070-197b4bc0eac9"
+			"8f771bdc-9258-42e8-a49f-fe34bbd360c4" "a6bf1ad2-37f3-46dc-8513-8c5aa5a9c501"
+		)
+	)
